File: ALIKEY03a.kicad_pcb (KiCad board)
At the start: 2 copper layers, 70 x 15 mm, 32 parts, among them J0 TestPoint, K1 B3W-9010-RG2N, K2 B3W-9010-RG2N, K3 B3W-9010-RG2N, P1 TestPoint, P2 TestPoint, P3 TestPoint

Commit message: Final version
Parts:
- D1-1, D1-2, D2-1, D2-2, D3-1, D3-2: footprint SMD_PAD_Generic:SMD_PAD_R200_508R50 -> Library:SMD_PAD_R200_508R50
- J0, P1, P2, P3: footprint SMD_PAD_Generic:SMD_PAD_R254_508R50 -> Library:SMD_PAD_R254_508R50
- K1, K2, K3: footprint THD_Switch_Omron:B3W-90xx-x2xN_Omron -> Library:B3W-90xx-x2xN_Omron
- R1, R10, R11, R12, R13, R14, R15, R2, R3, R4, R5, R6, R7, R8, R9: footprint SMD_Resistor_Generic:RESC3116X65N_1206 -> Library:RESC3116X65N_1206
- REF** (x4): footprint THD_Mechanical_Generic:MountingHole_3.2mm_M3 -> Library:MountingHole_3.2mm_M3
Other:
- board text added: "0.2032 mm / 0.2032 mm"
- board text added: "0.3048 mm"
- board text added: "1.6000 mm"
- board text added: "2"
- board text added: "70.0000 mm x 15.0000 mm"
- board text added: "BOARD CHARACTERISTICS"
- board text added: "BOT"
- board text added: "Board Thickness:"
- board text added: "Board overall dimensions:"
- board text added: "Castellated pads:"
- board text added: "Copper Finish:"
- board text added: "Copper Layer Count:"
- board text added: "Edge card connectors:"
- board text added: "HAL SnPb"
- board text added: "Impedance Control:"
- board text added: "Min hole diameter:"
- board text added: "Min track/spacing:"
- board text added: "No"
- board text added: "Plated Board Edge:"
- board text added: "TOP"
