File: ALIKEY03a.kicad_sch (KiCad schematic)
At the start: 28 parts, among them J0 TestPoint, K1 B3W-9010-RG2N, K2 B3W-9010-RG2N, K3 B3W-9010-RG2N, P1 TestPoint, P2 TestPoint, P3 TestPoint

Commit message: Final version
Parts:
- D1-1, D1-2, D2-1, D2-2, D3-1, D3-2, J0, P1, P2, P3: symbol Technology:TestPoint-PAD_THD_C250_250H80 -> Library:TestPoint-PAD_THD_C250_250H80
- K1, K2, K3: symbol Switch_Omron:B3W-9010-RG2N, PushButton, 2 LED -> Library:B3W-9010-RG2N, PushButton, 2 LED
- R1, R10, R11, R12, R13, R14, R15, R2, R3, R4, R5, R6, R7, R8, R9: symbol Resistor_SMD_1206_0.25W_1perc_Generic:2k2, SMD 1206, 0.25W, 1% -> Library:2k2, SMD 1206, 0.25W, 1%
Changed lines of the file:
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@@
 	(title_block
 		(title "ALIKEY03a - Tlacidlova doska 1x3")
-		(date "2024-10-23")
+		(date "2024-10-25")
 		(rev "00")
 		(company "VRM, a.s.")
 		(comment 1 "Janis Peter")
-		(comment 2 "www.zelektrik.sk")
-		(comment 3 "typename")
-		(comment 4 "c4")
-		(comment 5 "c5")
-		(comment 6 "c6")
-		(comment 7 "c7")
-		(comment 8 "c8")
-		(comment 9 "c9")
+		(comment 2 "www.vrm.sk")
 	)
 	(junction
@@
 	)
 	(symbol
-		(lib_id "Technology:TestPoint-PAD_THD_C250_250H80")
+		(lib_id "Library:TestPoint-PAD_THD_C250_250H80")
 		(at 64.77 35.56 90)
 		(unit 1)
@@
 	)
 	(symbol
-		(lib_id "Technology:TestPoint-PAD_THD_C250_250H80")
+		(lib_id "Library:TestPoint-PAD_THD_C250_250H80")
 		(at 138.43 92.71 270)
 		(unit 1)
@@
 	)
 	(symbol
-		(lib_id "Technology:TestPoint-PAD_THD_C250_250H80")
+		(lib_id "Library:TestPoint-PAD_THD_C250_250H80")
 		(at 158.75 92.71 270)
 		(unit 1)
@@
 	)
 	(symbol
-		(lib_id "Switch_Omron:B3W-9010-RG2N, PushButton, 2 LED")
+		(lib_id "Library:B3W-9010-RG2N, PushButton, 2 LED")
 		(at 50.8 63.5 0)
 		(unit 1)
@@
 	)
 	(symbol
-		(lib_id "_Symbol:GND_Bar")
+		(lib_id "Library:GND_Bar")
 		(at 40.64 67.31 0)
 		(unit 1)
@@
 	)
 	(symbol
-		(lib_id "Technology:TestPoint-PAD_THD_C250_250H80")
+		(lib_id "Library:TestPoint-PAD_THD_C250_250H80")
 		(at 50.8 92.71 270)
 		(unit 1)
@@
 	)
 	(symbol
-		(lib_id "Resistor_SMD_1206_0.25W_1perc_Generic:2k2, SMD 1206, 0.25W, 1%")
+		(lib_id "Library:2k2, SMD 1206, 0.25W, 1%")
 		(at 71.12 81.28 90)
 		(unit 1)
@@
 	)
 	(symbol
-		(lib_id "Technology:TestPoint-PAD_THD_C250_250H80")
+		(lib_id "Library:TestPoint-PAD_THD_C250_250H80")
 		(at 30.48 35.56 90)
 		(unit 1)
@@
 	)
 	(symbol
-		(lib_id "Resistor_SMD_1206_0.25W_1perc_Generic:2k2, SMD 1206, 0.25W, 1%")
+		(lib_id "Library:2k2, SMD 1206, 0.25W, 1%")
 		(at 109.22 81.28 90)
 		(unit 1)
@@
 	)
 	(symbol
-		(lib_id "Resistor_SMD_1206_0.25W_1perc_Generic:2k2, SMD 1206, 0.25W, 1%")
+		(lib_id "Library:2k2, SMD 1206, 0.25W, 1%")
 		(at 64.77 81.28 90)
 		(unit 1)
@@
 	)
 	(symbol
-		(lib_id "_Symbol:GND_Bar")
+		(lib_id "Library:GND_Bar")
 		(at 128.27 67.31 0)
 		(unit 1)
@@
 	)
 	(symbol
-		(lib_id "Resistor_SMD_1206_0.25W_1perc_Generic:2k2, SMD 1206, 0.25W, 1%")
+		(lib_id "Library:2k2, SMD 1206, 0.25W, 1%")
 		(at 109.22 48.26 90)
 		(unit 1)
@@
 	)
 	(symbol
-		(lib_id "Resistor_SMD_1206_0.25W_1perc_Generic:2k2, SMD 1206, 0.25W, 1%")
+		(lib_id "Library:2k2, SMD 1206, 0.25W, 1%")
 		(at 115.57 81.28 90)
 		(unit 1)
@@
 	)
 	(symbol
-		(lib_id "Resistor_SMD_1206_0.25W_1perc_Generic:2k2, SMD 1206, 0.25W, 1%")
+		(lib_id "Library:2k2, SMD 1206, 0.25W, 1%")
 		(at 152.4 48.26 90)
 		(unit 1)
@@
 	)
 	(symbol
-		(lib_id "Resistor_SMD_1206_0.25W_1perc_Generic:2k2, SMD 1206, 0.25W, 1%")
+		(lib_id "Library:2k2, SMD 1206, 0.25W, 1%")
 		(at 144.78 81.28 90)
 		(unit 1)
@@
 	)
 	(symbol
-		(lib_id "Technology:TestPoint-PAD_THD_C250_250H80")
+		(lib_id "Library:TestPoint-PAD_THD_C250_250H80")
 		(at 95.25 92.71 270)
 		(unit 1)
@@
 	)
 	(symbol
-		(lib_id "Resistor_SMD_1206_0.25W_1perc_Generic:2k2, SMD 1206, 0.25W, 1%")
+		(lib_id "Library:2k2, SMD 1206, 0.25W, 1%")
 		(at 57.15 81.28 90)
 		(unit 1)
@@
 	)
 	(symbol
-		(lib_id "Resistor_SMD_1206_0.25W_1perc_Generic:2k2, SMD 1206, 0.25W, 1%")
+		(lib_id "Library:2k2, SMD 1206, 0.25W, 1%")
 		(at 138.43 81.28 90)
 		(unit 1)
@@
 	)
 	(symbol
-		(lib_id "Technology:TestPoint-PAD_THD_C250_250H80")
+		(lib_id "Library:TestPoint-PAD_THD_C250_250H80")
 		(at 152.4 35.56 90)
 		(unit 1)
@@
 	)
 	(symbol
-		(lib_id "Resistor_SMD_1206_0.25W_1perc_Generic:2k2, SMD 1206, 0.25W, 1%")
+		(lib_id "Library:2k2, SMD 1206, 0.25W, 1%")
 		(at 101.6 81.28 90)
 		(unit 1)
@@
 	)
 	(symbol
-		(lib_id "Technology:TestPoint-PAD_THD_C250_250H80")
+		(lib_id "Library:TestPoint-PAD_THD_C250_250H80")
 		(at 115.57 92.71 270)
 		(unit 1)
@@
 	)
 	(symbol
-		(lib_id "_Symbol:GND_Bar")
+		(lib_id "Library:GND_Bar")
 		(at 30.48 38.1 0)
 		(unit 1)
@@
 	)
 	(symbol
-		(lib_id "Resistor_SMD_1206_0.25W_1perc_Generic:2k2, SMD 1206, 0.25W, 1%")
+		(lib_id "Library:2k2, SMD 1206, 0.25W, 1%")
 		(at 95.25 81.28 90)
 		(unit 1)
@@
 	)
 	(symbol
-		(lib_id "_Symbol:GND_Bar")
+		(lib_id "Library:GND_Bar")
 		(at 85.09 67.31 0)
 		(unit 1)
@@
 	)
 	(symbol
-		(lib_id "Resistor_SMD_1206_0.25W_1perc_Generic:2k2, SMD 1206, 0.25W, 1%")
+		(lib_id "Library:2k2, SMD 1206, 0.25W, 1%")
 		(at 158.75 81.28 90)
 		(unit 1)
@@
 	)
 	(symbol
-		(lib_id "Switch_Omron:B3W-9010-RG2N, PushButton, 2 LED")
+		(lib_id "Library:B3W-9010-RG2N, PushButton, 2 LED")
 		(at 95.25 63.5 0)
 		(unit 1)
@@
 	)
 	(symbol
-		(lib_id "Resistor_SMD_1206_0.25W_1perc_Generic:2k2, SMD 1206, 0.25W, 1%")
+		(lib_id "Library:2k2, SMD 1206, 0.25W, 1%")
 		(at 152.4 81.28 90)
 		(unit 1)
@@
 	)
 	(symbol
-		(lib_id "Resistor_SMD_1206_0.25W_1perc_Generic:2k2, SMD 1206, 0.25W, 1%")
+		(lib_id "Library:2k2, SMD 1206, 0.25W, 1%")
 		(at 64.77 48.26 90)
 		(unit 1)
@@
 	)
 	(symbol
-		(lib_id "Technology:TestPoint-PAD_THD_C250_250H80")
+		(lib_id "Library:TestPoint-PAD_THD_C250_250H80")
 		(at 71.12 92.71 270)
 		(unit 1)
@@
 	)
 	(symbol
-		(lib_id "Switch_Omron:B3W-9010-RG2N, PushButton, 2 LED")
+		(lib_id "Library:B3W-9010-RG2N, PushButton, 2 LED")
 		(at 138.43 63.5 0)
 		(unit 1)
@@
 	)
 	(symbol
-		(lib_id "Resistor_SMD_1206_0.25W_1perc_Generic:2k2, SMD 1206, 0.25W, 1%")
+		(lib_id "Library:2k2, SMD 1206, 0.25W, 1%")
 		(at 50.8 81.28 90)
 		(unit 1)
@@
 	)
 	(symbol
-		(lib_id "Technology:TestPoint-PAD_THD_C250_250H80")
+		(lib_id "Library:TestPoint-PAD_THD_C250_250H80")
 		(at 109.22 35.56 90)
 		(unit 1)
